Commit message: ignored rplidar_ros

File: robot_model/urdf/robot_model.urdf.xacro (robot description, xacro)
@@ -1,6 +1,7 @@
 <?xml version="1.0"?>
 <robot xmlns:xacro="http://www.ros.org/wiki/xacro" name="tour_guide_robot">
+  <!--
     <xacro:include filename="$(find robot_model)/urdf/gazebo_config.xacro" />
-    <xacro:include filename="$(find robot_model)/urdf/robot_plugins.gazebo" />
+    <xacro:include filename="$(find robot_model)/urdf/robot_plugins.gazebo" /> -->
     <!-- Material : colors -->
     <material name="red">
@@ -14,5 +15,5 @@
     </material>
     <!-- ################################# -->
-    <!-- base link  -->
+    <!-- base link -->
     <link name="base_footprint" />
     <!-- Chassis link -->
@@ -127,5 +128,5 @@
    </joint>
    <!-- lider link -->
-   <link name="lidar_link">
+   <link name="laser_link">
     <inertial>
         <origin xyz="0.0 0.0 0.0" rpy="0.0 0.0 0.0"/>
@@ -151,5 +152,5 @@
         <origin xyz="0.2 0.0 0.07" rpy="0.0 0.0 0.0"/>
         <parent link="chassis_link"/>
-        <child link="lidar_link"/>
+        <child link="laser_link"/>
     </joint>
 </robot>
